Commit message: Adjust offset position/angle of camera_link and camera_usb_plug_link

File: realsense2_description/urdf/_d435.urdf.xacro (robot description, xacro)
@@ -135,5 +135,5 @@
     <xacro:if value="${add_plug}">
       <xacro:usb_plug parent="${name}_link" name="${name}_usb_plug">
-        <origin xyz="${d435_cam_mount_from_center_offset - 0.02095} ${-d435_cam_depth_py - 0.0353} 0" rpy="0 0 0"/>
+        <origin xyz="${d435_cam_mount_from_center_offset - 0.0315} ${-d435_cam_depth_py - 0.0353} 0" rpy="0 0 0"/>
       </xacro:usb_plug>
     </xacro:if>

File: realsense2_description/urdf/xarm_d435_camera.urdf.xacro (robot description, xacro)
@@ -8,5 +8,5 @@
   <xacro:include filename="$(find realsense2_description)/urdf/_d435.urdf.xacro" />
   <xacro:sensor_d435 parent="$(arg prefix)link_eef" use_nominal_extrinsics="$(arg use_nominal_extrinsics)" add_plug="$(arg add_plug)" use_mesh="$(arg use_mesh)" topics_ns="$(arg topics_ns)" publish_pointcloud="$(arg publish_pointcloud)" >
-    <origin xyz="0.075 0 0.012" rpy="0 ${-pi/2} 0"/>
+    <origin xyz="0.055 0 0.012" rpy="0 ${-pi/2} ${pi}"/>
   </xacro:sensor_d435>
 </robot>
